Commit message: New version
Has rtabmap and fixed odom and tf

File: src/project/urdf/quad.urdf.xacro (robot description, xacro)
@@ -1,98 +1,186 @@
 <?xml version="1.0"?>
 <robot xmlns:xacro="http://ros.org/wiki/xacro" name="quad">
-  <!-- Arguments -->
-  <xacro:arg name="use_ros2_control" default="true"/>
-  <!-- ====================== BASE BOX ====================== -->
+  <!-- PROPERTIES -->
+  <xacro:property name="chassis_length" value="0.4" />
+  <xacro:property name="chassis_width" value="0.3" />
+  <xacro:property name="chassis_height" value="0.1" />
+  <xacro:property name="chassis_mass" value="5.0" />
+  <xacro:property name="wheel_radius" value="0.05" />
+  <xacro:property name="wheel_thickness" value="0.04" />
+  <xacro:property name="wheel_mass" value="0.5" />
+  <xacro:property name="wheel_y_offset" value="${chassis_width / 2 + wheel_thickness / 2}" />
+  <xacro:property name="caster_radius" value="0.025" />
+  <xacro:property name="caster_mass" value="0.1" />
+  <xacro:property name="M_PI" value="3.1415926535897931" />
+  <!-- INERTIA MACROS -->
+  <xacro:macro name="box_inertia" params="m w h d">
+    <inertial>
+      <mass value="${m}"/>
+      <inertia ixx="${(m/12)*(h*h+d*d)}" ixy="0" ixz="0"
+               iyy="${(m/12)*(w*w+d*d)}" iyz="0"
+               izz="${(m/12)*(w*w+h*h)}"/>
+    </inertial>
+  </xacro:macro>
+  <xacro:macro name="cylinder_inertia" params="m r h">
+    <inertial>
+      <mass value="${m}"/>
+      <inertia ixx="${(m/12)*(3*r*r+h*h)}" ixy="0" ixz="0"
+               iyy="${(m/12)*(3*r*r+h*h)}" iyz="0"
+               izz="${m*r*r/2}"/>
+    </inertial>
+  </xacro:macro>
+  <xacro:macro name="sphere_inertia" params="m r">
+    <inertial>
+      <mass value="${m}"/>
+      <inertia ixx="${2*m*r*r/5}" ixy="0" ixz="0"
+               iyy="${2*m*r*r/5}" iyz="0"
+               izz="${2*m*r*r/5}"/>
+    </inertial>
+  </xacro:macro>
+  <!-- BASE LINK -->
   <link name="base_link">
     <visual>
-      <origin xyz="0 0 0.05" rpy="0 0 0"/>
+      <geometry><box size="${chassis_length} ${chassis_width} ${chassis_height}"/></geometry>
+      <material name="blue"><color rgba="0.0 0.0 1.0 1.0"/></material>
+    </visual>
+    <collision>
+      <geometry><box size="${chassis_length} ${chassis_width} ${chassis_height}"/></geometry>
+    </collision>
+    <xacro:box_inertia m="${chassis_mass}" w="${chassis_length}" h="${chassis_width}" d="${chassis_height}"/>
+  </link>
+  <!-- CASTER WHEEL -->
+  <link name="caster_wheel_link">
+    <visual>
+      <geometry><sphere radius="${caster_radius}"/></geometry>
+      <material name="grey"><color rgba="0.5 0.5 0.5 1.0"/></material>
+    </visual>
+    <collision>
+      <geometry><sphere radius="${caster_radius}"/></geometry>
+    </collision>
+    <xacro:sphere_inertia m="${caster_mass}" r="${caster_radius}"/>
+  </link>
+  <joint name="caster_wheel_joint" type="fixed">
+    <parent link="base_link"/>
+    <child link="caster_wheel_link"/>
+    <origin xyz="${chassis_length/2 - caster_radius} 0 ${-(chassis_height/2) - wheel_radius + caster_radius*2}" rpy="0 0 0"/>
+  </joint>
+  <!-- LEFT WHEEL -->
+  <link name="left_wheel_link">
+    <visual>
+      <origin xyz="0 0 0" rpy="${M_PI/2} 0 0"/>
       <geometry>
-        <box size="0.5 0.5 0.1"/> <!-- 50cm x 50cm x 10cm -->
+        <cylinder radius="${wheel_radius}" length="${wheel_thickness}"/>
       </geometry>
-      <material name="blue">
-        <color rgba="0 0 1 1"/>
+      <material name="black">
+        <color rgba="0.1 0.1 0.1 1.0"/>
       </material>
     </visual>
     <collision>
-      <origin xyz="0 0 0.05" rpy="0 0 0"/>
+      <origin xyz="0 0 0" rpy="${M_PI/2} 0 0"/>
       <geometry>
-        <box size="0.5 0.5 0.1"/>
+        <cylinder radius="${wheel_radius}" length="${wheel_thickness}"/>
       </geometry>
     </collision>
-    <inertial>
-      <origin xyz="0 0 0.05" rpy="0 0 0"/>
-      <mass value="2.0"/>
-      <inertia ixx="0.0833" ixy="0" ixz="0"
-               iyy="0.0833" iyz="0"
-               izz="0.125"/>
-    </inertial>
+    <xacro:cylinder_inertia m="${wheel_mass}" r="${wheel_radius}" h="${wheel_thickness}"/>
   </link>
-  <!-- ====================== LIDAR MOUNT ====================== -->
-  <link name="lidar_link">
+  <joint name="left_wheel_joint" type="continuous">
+    <parent link="base_link"/>
+    <child link="left_wheel_link"/>
+    <origin xyz="0 ${wheel_y_offset} ${-(chassis_height/2)}" rpy="0 0 0"/>
+    <axis xyz="0 1 0"/>
+  </joint>
+  <!-- RIGHT WHEEL -->
+  <link name="right_wheel_link">
     <visual>
-      <origin xyz="0 0 0.05" rpy="0 0 0"/>
+      <origin xyz="0 0 0" rpy="${M_PI/2} 0 0"/>
       <geometry>
-        <cylinder radius="0.05" length="0.1"/>
+        <cylinder radius="${wheel_radius}" length="${wheel_thickness}"/>
       </geometry>
       <material name="black">
-        <color rgba="0.1 0.1 0.1 1"/>
+        <color rgba="0.1 0.1 0.1 1.0"/>
       </material>
     </visual>
     <collision>
-      <origin xyz="0 0 0.05" rpy="0 0 0"/>
+      <origin xyz="0 0 0" rpy="${M_PI/2} 0 0"/>
       <geometry>
-        <cylinder radius="0.05" length="0.1"/>
+        <cylinder radius="${wheel_radius}" length="${wheel_thickness}"/>
       </geometry>
     </collision>
-    <inertial>
-      <mass value="0.5"/>
-      <inertia ixx="0.001" ixy="0" ixz="0" iyy="0.001" iyz="0" izz="0.001"/>
-    </inertial>
+    <xacro:cylinder_inertia m="${wheel_mass}" r="${wheel_radius}" h="${wheel_thickness}"/>
   </link>
-  <!-- Joint: lidar mounted 0.2m above box center -->
-  <joint name="base_to_lidar" type="fixed">
+  <joint name="right_wheel_joint" type="continuous">
+    <parent link="base_link"/>
+    <child link="right_wheel_link"/>
+    <origin xyz="0 ${-wheel_y_offset} ${-(chassis_height/2)}" rpy="0 0 0"/>
+    <axis xyz="0 1 0"/>
+  </joint>
+  <!-- LIDAR -->
+  <link name="lidar_link">
+    <visual>
+      <geometry><cylinder radius="0.05" length="0.1"/></geometry>
+      <material name="black"/>
+    </visual>
+    <collision>
+      <geometry><cylinder radius="0.05" length="0.1"/></geometry>
+    </collision>
+    <xacro:cylinder_inertia m="0.1" r="0.05" h="0.1"/>
+  </link>
+  <joint name="lidar_joint" type="fixed">
     <parent link="base_link"/>
     <child link="lidar_link"/>
-    <origin xyz="0 0 0.15" rpy="0 0 0"/>
+    <origin xyz="0 0 ${chassis_height/2 + 0.05}" rpy="0 0 0"/>
   </joint>
-  <!-- ====================== GAZEBO PLUGIN: 3D LIDAR ====================== -->
- <gazebo reference="lidar_link">
-  <sensor name="lidar" type="gpu_lidar">
-    <always_on>true</always_on>
-    <visualize>true</visualize>
-    <update_rate>10</update_rate>
-    <pose>0 0 0 0 0 0</pose>
-    <lidar>
-      <scan>
-        <horizontal>
-          <samples>360</samples>
-          <resolution>1</resolution>
-          <min_angle>-3.14159</min_angle>
-          <max_angle>3.14159</max_angle>
-        </horizontal>
-        <vertical>
-          <samples>10</samples>
-          <resolution>1</resolution>
-          <min_angle>-0.2618</min_angle> <!-- -15 degrees -->
-          <max_angle>0.2618</max_angle> <!-- 15 degrees -->
-        </vertical>
-      </scan>
-      <range>
-        <min>0.12</min>
-        <max>30.0</max>
-        <resolution>0.01</resolution>
-      </range>
-      <noise>
-        <type>gaussian</type>
-        <mean>0.0</mean>
-        <stddev>0.01</stddev>
-      </noise>
-      <enable_intensity>false</enable_intensity>
-    </lidar>
-   <output_type>points</output_type>
-    <!-- Topic and frame -->
-    <topic>/scan</topic>
-    <frame_id>lidar_link</frame_id>
-  </sensor>
- </gazebo>
+  <gazebo reference="lidar_link">
+    <sensor name="lidar" type="gpu_lidar">
+      <always_on>true</always_on>
+      <update_rate>10</update_rate>
+      <topic>/scan</topic>
+      <frame_id>lidar_link</frame_id>
+      <lidar>
+        <scan>
+          <horizontal>
+            <samples>720</samples>
+            <resolution>1</resolution>
+            <min_angle>-3.14159</min_angle>
+            <max_angle>3.14159</max_angle>
+          </horizontal>
+          <vertical>
+            <samples>16</samples>
+            <resolution>1</resolution>
+            <min_angle>-0.2618</min_angle>
+            <max_angle>0.2618</max_angle>
+          </vertical>
+        </scan>
+        <range>
+          <min>0.12</min>
+          <max>30.0</max>
+          <resolution>0.01</resolution>
+        </range>
+        <noise>
+          <type>gaussian</type>
+          <mean>0.0</mean>
+          <stddev>0.01</stddev>
+        </noise>
+      </lidar>
+      <output_type>points</output_type>
+    </sensor>
+  </gazebo>
+  <gazebo>
+    <plugin name="gz::sim::systems::DiffDrive" filename="gz-sim-diff-drive-system">
+      <left_joint>left_wheel_joint</left_joint>
+      <right_joint>right_wheel_joint</right_joint>
+      <wheel_separation>${wheel_y_offset * 2}</wheel_separation>
+      <wheel_radius>${wheel_radius}</wheel_radius>
+      <odom_publish_frequency>50</odom_publish_frequency>
+      <topic>cmd_vel</topic>
+      <frame_id>odom</frame_id>
+      <child_frame_id>base_link</child_frame_id>
+    </plugin>
+  </gazebo>
+  <gazebo>
+    <plugin name="gz::sim::systems::JointStatePublisher" filename="gz-sim-joint-state-publisher-system">
+      <joint_name>left_wheel_joint</joint_name>
+      <joint_name>right_wheel_joint</joint_name>
+    </plugin>
+  </gazebo>
 </robot>
