Commit message: Added Camera

File: src/project/urdf/quadped.urdf (robot description, URDF)
Before this commit: robot quadped, 113 links, 112 joints
Links:
- added link Camera_link; visual cylinder length=0.00741 radius=0.01355
Joints:
- added joint Camera_link_joint: type fixed, parent baselink_link, child Camera_link, origin xyz=0.05046 -0.18221 0.00592 rpy=1.57080 -1.57080 0.00000

Commit message: Tried to add movement

File: src/project/urdf/quadped.urdf (robot description, URDF)
Before this commit: robot quadped, 114 links, 113 joints
Joints:
- joint blhipmotorplate_link_joint: limit effort=100.00000 velocity=10.0 -> effort=100.00000 velocity=2.0
- joint blpart1_link_joint: limit effort=100.00000 velocity=10.0 -> effort=100.00000 velocity=2.0; origin xyz=-0.01314 -0.04226 -0.00388 rpy=-0.00000 -1.57080 0.00000 -> xyz=0.01425 -0.00052 0.00006 rpy=-0.00000 -1.57080 0.00000; parent blupperleg_link -> bllowerlegmotor_link
- joint blpart5_link_joint: limit effort=100.00000 velocity=10.0 -> effort=100.00000 velocity=2.0
- joint blpin1_link_joint: limit effort=100.00000 velocity=10.0 -> effort=100.00000 velocity=2.0
- joint blpin3_link_joint: limit effort=100.00000 velocity=10.0 -> effort=100.00000 velocity=2.0
- joint blpin5_link_joint: limit effort=100.00000 velocity=10.0 -> effort=100.00000 velocity=2.0
- joint blupperlegmotorplate_link_joint: limit effort=100.00000 velocity=10.0 -> effort=100.00000 velocity=2.0
- joint brhipmotorplate_link_joint: limit effort=100.00000 velocity=10.0 -> effort=100.00000 velocity=2.0
- joint brpart1_link_joint: limit effort=100.00000 velocity=10.0 -> effort=100.00000 velocity=2.0; origin xyz=0.01314 -0.04234 -0.00394 rpy=-0.00000 1.57080 0.00000 -> xyz=-0.01425 -0.00060 -0.00000 rpy=0.00000 1.57080 0.00000; parent brupperleg_link -> brlowerlegmotor_link
- joint brpart5_link_joint: limit effort=100.00000 velocity=10.0 -> effort=100.00000 velocity=2.0
- joint brpin1_link_joint: limit effort=100.00000 velocity=10.0 -> effort=100.00000 velocity=2.0
- joint brpin3_link_joint: limit effort=100.00000 velocity=0.00000 -> effort=100.00000 velocity=2.0
- joint brpin5_link_joint: limit effort=100.00000 velocity=10.0 -> effort=100.00000 velocity=2.0
- joint brupperlegmotoplate_link_joint: limit effort=100.00000 velocity=10.0 -> effort=100.00000 velocity=2.0
- joint flhipmotorplate_link_joint: limit effort=100.00000 velocity=10.0 -> effort=100.00000 velocity=2.0
- joint flpart1_link_joint: limit effort=100.00000 velocity=10.0 -> effort=100.00000 velocity=2.0; origin xyz=-0.01314 -0.04236 -0.00393 rpy=0.00000 -1.57080 0.00000 -> xyz=0.01425 -0.00061 0.00001 rpy=0.00000 -1.57080 0.00000; parent flupperleg_link -> fllowerlegmotor_link
- joint flpart5_link_joint: limit effort=100.00000 velocity=10.0 -> effort=100.00000 velocity=2.0
- joint flpin1_link_joint: limit effort=100.00000 velocity=10.0 -> effort=100.00000 velocity=2.0
- joint flpin3_link_joint: limit effort=100.00000 velocity=10.0 -> effort=100.00000 velocity=2.0
- joint flpin5_link_joint: limit effort=100.00000 velocity=10.0 -> effort=100.00000 velocity=2.0
- joint flupperlegmotorplate_link_joint: limit effort=100.00000 velocity=10.0 -> effort=100.00000 velocity=2.0
- joint frhipmotorplate_link_joint: limit effort=100.00000 velocity=10.0 -> effort=100.00000 velocity=2.0
- joint frpart1_link_joint: limit effort=100.00000 velocity=10.0 -> effort=100.00000 velocity=2.0; origin xyz=0.01314 -0.04227 -0.00397 rpy=0.00000 1.57080 0.00000 -> xyz=-0.01425 -0.00052 -0.00003 rpy=0.00000 1.57080 0.00000; parent frupperleg_link -> frlowerlegmotor_link
- joint frpart5_link_joint: limit effort=100.00000 velocity=10.0 -> effort=100.00000 velocity=2.0
- joint frpin1_link_joint: limit effort=100.00000 velocity=10.0 -> effort=100.00000 velocity=2.0
- joint frpin3_link_joint: limit effort=100.00000 velocity=10.0 -> effort=100.00000 velocity=2.0
- joint frpin5_link_joint: limit effort=100.00000 velocity=10.0 -> effort=100.00000 velocity=2.0
- joint frupperlegmotorplate_link_joint: limit effort=100.00000 velocity=10.0 -> effort=100.00000 velocity=2.0

Commit message: Fixed Cam orientation in urdf

File: src/project/urdf/quadped.urdf (robot description, URDF)
Before this commit: robot quadped, 114 links, 113 joints
Links:
- added link Camera_link_optical
Joints:
- added joint Camera_link_optical_joint: type fixed, parent Camera_link, child Camera_link_optical, origin xyz=0 0 0 rpy=-1.5708 -1.5708 -1.5708

Commit message: Trying to write scripts

File: src/project/urdf/quadped.urdf (robot description, URDF)
Before this commit: robot quadped, 115 links, 114 joints
Joints:
- joint blhipmotorplate_link_joint: limit effort=100.00000 velocity=2.0 -> lower=-3.14000 upper=3.14000 effort=100.00000 velocity=10.00000; type continuous -> revolute
- joint blpart1_link_joint: limit effort=100.00000 velocity=2.0 -> lower=-3.14000 upper=3.14000 effort=100.00000 velocity=10.00000; type continuous -> revolute
- joint blpart5_link_joint: limit effort=100.00000 velocity=2.0 -> lower=-3.14000 upper=3.14000 effort=100.00000 velocity=10.00000; type continuous -> revolute
- joint blpin1_link_joint: limit effort=100.00000 velocity=2.0 -> lower=-3.14000 upper=3.14000 effort=100.00000 velocity=10.00000; type continuous -> revolute
- joint blpin3_link_joint: limit effort=100.00000 velocity=2.0 -> lower=-3.14000 upper=3.14000 effort=100.00000 velocity=10.00000; type continuous -> revolute
- joint blpin5_link_joint: limit effort=100.00000 velocity=2.0 -> lower=-3.14000 upper=3.14000 effort=100.00000 velocity=10.00000; type continuous -> revolute
- joint blupperlegmotorplate_link_joint: limit effort=100.00000 velocity=2.0 -> lower=-3.14000 upper=3.14000 effort=100.00000 velocity=10.00000; type continuous -> revolute
- joint brhipmotorplate_link_joint: limit effort=100.00000 velocity=2.0 -> lower=-3.14000 upper=3.14000 effort=100.00000 velocity=10.00000; type continuous -> revolute
- joint brpart1_link_joint: limit effort=100.00000 velocity=2.0 -> lower=-3.14000 upper=3.14000 effort=100.00000 velocity=10.00000; type continuous -> revolute
- joint brpart5_link_joint: limit effort=100.00000 velocity=2.0 -> lower=-3.14000 upper=3.14000 effort=100.00000 velocity=10.00000; type continuous -> revolute
- joint brpin1_link_joint: limit effort=100.00000 velocity=2.0 -> lower=-3.14000 upper=3.14000 effort=100.00000 velocity=10.00000; type continuous -> revolute
- joint brpin3_link_joint: limit effort=100.00000 velocity=2.0 -> lower=-3.14000 upper=3.14000 effort=100.00000 velocity=10.00000; type continuous -> revolute
- joint brpin5_link_joint: limit effort=100.00000 velocity=2.0 -> lower=-3.14000 upper=3.14000 effort=100.00000 velocity=10.00000; type continuous -> revolute
- joint brupperlegmotoplate_link_joint: limit effort=100.00000 velocity=2.0 -> lower=-3.14000 upper=3.14000 effort=100.00000 velocity=10.00000; type continuous -> revolute
- joint flhipmotorplate_link_joint: limit effort=100.00000 velocity=2.0 -> lower=-3.14000 upper=3.14000 effort=100.00000 velocity=10.00000; type continuous -> revolute
- joint flpart1_link_joint: limit effort=100.00000 velocity=2.0 -> lower=-3.14000 upper=3.14000 effort=100.00000 velocity=10.00000; type continuous -> revolute
- joint flpart5_link_joint: limit effort=100.00000 velocity=2.0 -> lower=-3.14000 upper=3.14000 effort=100.00000 velocity=10.00000; type continuous -> revolute
- joint flpin1_link_joint: limit effort=100.00000 velocity=2.0 -> lower=-3.14000 upper=3.14000 effort=100.00000 velocity=10.00000; type continuous -> revolute
- joint flpin3_link_joint: limit effort=100.00000 velocity=2.0 -> lower=-3.14000 upper=3.14000 effort=100.00000 velocity=10.00000; type continuous -> revolute
- joint flpin5_link_joint: limit effort=100.00000 velocity=2.0 -> lower=-3.14000 upper=3.14000 effort=100.00000 velocity=10.00000; type continuous -> revolute
- joint flupperlegmotorplate_link_joint: limit effort=100.00000 velocity=2.0 -> lower=-3.14000 upper=3.14000 effort=100.00000 velocity=10.00000; type continuous -> revolute
- joint frhipmotorplate_link_joint: limit effort=100.00000 velocity=2.0 -> lower=-3.14000 upper=3.14000 effort=100.00000 velocity=10.00000; type continuous -> revolute
- joint frpart1_link_joint: limit effort=100.00000 velocity=2.0 -> lower=-3.14000 upper=3.14000 effort=100.00000 velocity=10.00000; type continuous -> revolute
- joint frpart5_link_joint: limit effort=100.00000 velocity=2.0 -> lower=-3.14000 upper=3.14000 effort=100.00000 velocity=10.00000; type continuous -> revolute
- joint frpin1_link_joint: limit effort=100.00000 velocity=2.0 -> lower=-3.14000 upper=3.14000 effort=100.00000 velocity=10.00000; type continuous -> revolute
- joint frpin3_link_joint: limit effort=100.00000 velocity=2.0 -> lower=-3.14000 upper=3.14000 effort=100.00000 velocity=10.00000; type continuous -> revolute
- joint frpin5_link_joint: limit effort=100.00000 velocity=2.0 -> lower=-3.14000 upper=3.14000 effort=100.00000 velocity=10.00000; type continuous -> revolute
- joint frupperlegmotorplate_link_joint: limit effort=100.00000 velocity=2.0 -> lower=-3.14000 upper=3.14000 effort=100.00000 velocity=10.00000; type continuous -> revolute

Commit message: Fixes

File: src/project/urdf/quadped.urdf (robot description, URDF)
Before this commit: robot quadped, 115 links, 114 joints
Links:
- added link IMU_link
Joints:
- added joint IMU_link_joint: type fixed, parent baselink_link, child IMU_link, origin xyz=0.04940 0.00032 0.04152 rpy=0.00000 0.00000 0.00000
- joint brpart5_link_joint: mimic joint=brpart1_link_joint multiplier=1.0 offset=0.0 -> joint=brpart1_link_joint multiplier=0.5 offset=0.0
